Commit message: Updates naming of package.

File: turtlelib/urdf/turtlebot3_burger.urdf.xacro (robot description, xacro)
@@ -2,5 +2,5 @@
 <robot name="turtlebot3_burger" xmlns:xacro="http://ros.org/wiki/xacro">
   <xacro:arg name="color" default="light_black" />
-  <xacro:property name="yaml_file" value="$(find turtle_description)/config/diff_params.yaml" />
+  <xacro:property name="yaml_file" value="$(find turtlelib)/config/diff_params.yaml" />
   <xacro:property name="diff_params" value="${xacro.load_yaml(yaml_file)}"/>
   <xacro:property name="track_width" value="${diff_params['track_width']}" />
@@ -49,5 +49,5 @@
       <origin xyz="-0.032 0 0.0" rpy="0 0 0"/>
       <geometry>
-        <mesh filename="package://turtle_description/meshes/burger_base.stl" scale="0.001 0.001 0.001"/>
+        <mesh filename="package://turtlelib/meshes/burger_base.stl" scale="0.001 0.001 0.001"/>
       </geometry>
         <material name="$(arg color)"/>
@@ -75,5 +75,5 @@
       <origin xyz="0 0 0" rpy="1.57 0 0"/>
       <geometry>
-        <mesh filename="package://turtle_description/meshes/left_tire.stl" scale="0.001 0.001 0.001"/>
+        <mesh filename="package://turtlelib/meshes/left_tire.stl" scale="0.001 0.001 0.001"/>
       </geometry>
       <material name="dark"/>
@@ -101,5 +101,5 @@
       <origin xyz="0 0 0" rpy="1.57 0 0"/>
       <geometry>
-        <mesh filename="package://turtle_description/meshes/right_tire.stl" scale="0.001 0.001 0.001"/>
+        <mesh filename="package://turtlelib/meshes/right_tire.stl" scale="0.001 0.001 0.001"/>
       </geometry>
       <material name="dark"/>
@@ -150,5 +150,5 @@
       <origin xyz="0 0 0.0" rpy="0 0 0"/>
       <geometry>
-	      <mesh filename="package://turtle_description/meshes/lds.stl" scale="0.001 0.001 0.001"/>
+	      <mesh filename="package://turtlelib/meshes/lds.stl" scale="0.001 0.001 0.001"/>
       </geometry>
       <material name="dark"/>
